File: samd51j18a/samd51j18a.kicad_pcb (KiCad board)
At the start: 2 copper layers, 72.4 x 26.7 mm, 35 parts, among them J1 Conn_01x20_Male, J4 Conn_01x20_Male, U1 ATSAMD51J18A-A, U2 NJM2866F33, Y1 32.768kHz

Commit message: finished samd21 dev board (syzygy), exported gerbers and drill files
Other:
- board text added: "BUNNY"
- board text added: "HOP"
Changed lines of the file:
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@@
   (general
     (thickness 1.6)
-    (drawings 46)
+    (drawings 48)
     (tracks 632)
     (zones 0)
@@
     (pcbplotparams
       (layerselection 0x010fc_ffffffff)
-      (usegerberextensions false)
+      (usegerberextensions true)
       (usegerberattributes true)
       (usegerberadvancedattributes true)
@@
       (plotinvisibletext false)
       (padsonsilk false)
-      (subtractmaskfromsilk false)
+      (subtractmaskfromsilk true)
       (outputformat 1)
       (mirror false)
-      (drillshape 1)
+      (drillshape 0)
       (scaleselection 1)
-      (outputdirectory ""))
+      (outputdirectory "gerbers/"))
   )
   (net 0 "")
@@
       (effects (font (size 1 1) (thickness 0.15)))
     )
-    (fp_text user %R (at 0 24.13) (layer F.Fab)
-      (effects (font (size 1 1) (thickness 0.15)))
-    )
     (fp_line (start -0.635 -1.27) (end 1.27 -1.27) (layer F.Fab) (width 0.1))
     (fp_line (start 1.27 -1.27) (end 1.27 49.53) (layer F.Fab) (width 0.1))
@@
     (fp_line (start 1.8 50.05) (end 1.8 -1.8) (layer F.CrtYd) (width 0.05))
     (fp_line (start 1.8 -1.8) (end -1.8 -1.8) (layer F.CrtYd) (width 0.05))
+    (fp_text user %R (at 0 24.13) (layer F.Fab)
+      (effects (font (size 1 1) (thickness 0.15)))
+    )
     (pad 20 thru_hole oval (at 0 48.26 90) (size 1.7 1.7) (drill 1) (layers *.Cu *.Mask)
       (net 15 PA19))
@@
       (effects (font (size 1 1) (thickness 0.15)))
     )
-    (fp_text user %R (at 0 24.13) (layer F.Fab)
-      (effects (font (size 1 1) (thickness 0.15)))
-    )
     (fp_line (start -0.635 -1.27) (end 1.27 -1.27) (layer F.Fab) (width 0.1))
     (fp_line (start 1.27 -1.27) (end 1.27 49.53) (layer F.Fab) (width 0.1))
@@
     (fp_line (start 1.8 50.05) (end 1.8 -1.8) (layer F.CrtYd) (width 0.05))
     (fp_line (start 1.8 -1.8) (end -1.8 -1.8) (layer F.CrtYd) (width 0.05))
+    (fp_text user %R (at 0 24.13) (layer F.Fab)
+      (effects (font (size 1 1) (thickness 0.15)))
+    )
     (pad 20 thru_hole oval (at 0 48.26 90) (size 1.7 1.7) (drill 1) (layers *.Cu *.Mask)
       (net 5 +3V3))
@@
     )
   )
+  (gr_text HOP (at 108.712 83.693) (layer B.SilkS)
+    (effects (font (size 4 4) (thickness 0.5)) (justify mirror))
+  )
+  (gr_text BUNNY (at 123.444 73.787) (layer B.SilkS)
+    (effects (font (size 4 4) (thickness 0.5)) (justify mirror))
+  )
   (dimension 11.938676 (width 0.15) (layer Dwgs.User)
     (gr_text "11.939 mm" (at 106.990016 83.062975 359.3904934) (layer Dwgs.User)
@@
   (gr_line (start 173.355 88.265) (end 173.355 61.595) (layer Edge.Cuts) (width 0.05))
   (gr_line (start 100.965 61.595) (end 173.355 61.595) (layer Edge.Cuts) (width 0.05))
-  (via (at 164.719 79.6925) (size 0.8) (drill 0.4) (layers F.Cu B.Cu) (net 39))
-  (via (at 165.862 79.6925) (size 0.8) (drill 0.4) (layers F.Cu B.Cu) (net 38))
-  (via (at 167.0685 79.6925) (size 0.8) (drill 0.4) (layers F.Cu B.Cu) (net 36))
-  (via (at 166.3065 75.438) (size 0.8) (drill 0.4) (layers F.Cu B.Cu) (net 36))
-  (via (at 165.354 71.0565) (size 0.8) (drill 0.4) (layers F.Cu B.Cu) (net 38))
-  (via (at 164.1475 70.0405) (size 0.8) (drill 0.4) (layers F.Cu B.Cu) (net 39))
-  (via (at 140.7795 78.74) (size 0.8) (drill 0.4) (layers F.Cu B.Cu) (net 35))
-  (via (at 136.779 78.9305) (size 0.8) (drill 0.4) (layers F.Cu B.Cu) (net 39))
-  (via (at 136.9695 82.169) (size 0.8) (drill 0.4) (layers F.Cu B.Cu) (net 38))
-  (via (at 135.763 82.042) (size 0.8) (drill 0.4) (layers F.Cu B.Cu) (net 36))
-  (via (at 138.2395 78.9305) (size 0.8) (drill 0.4) (layers F.Cu B.Cu) (net 34))
-  (via (at 142.6845 70.612) (size 0.8) (drill 0.4) (layers F.Cu B.Cu) (net 6))
-  (via (at 152.781 72.136) (size 0.8) (drill 0.4) (layers F.Cu B.Cu) (net 5))
   (via (at 152.781 73.406) (size 0.8) (drill 0.4) (layers F.Cu B.Cu) (net 1))
   (segment (start 125.73 70.0125) (end 127.028 70.0125) (width 0.25) (layer F.Cu) (net 1))
@@
   (segment (start 133.06899 71.59151) (end 133.717308 71.59151) (width 0.25) (layer F.Cu) (net 4))
   (segment (start 133.717308 71.59151) (end 134.6835 71.59151) (width 0.25) (layer F.Cu) (net 4))
+  (via (at 152.781 72.136) (size 0.8) (drill 0.4) (layers F.Cu B.Cu) (net 5))
   (via (at 108.331 67.31) (size 0.8) (drill 0.4) (layers F.Cu B.Cu) (net 5))
   (segment (start 120.114 67.945) (end 120.114 69.568) (width 0.25) (layer F.Cu) (net 5))
@@
   (segment (start 151.13 73.66) (end 152.654 72.136) (width 0.25) (layer B.Cu) (net 5))
   (segment (start 151.13 76.5175) (end 151.13 73.66) (width 0.25) (layer B.Cu) (net 5))
+  (via (at 142.6845 70.612) (size 0.8) (drill 0.4) (layers F.Cu B.Cu) (net 6))
   (segment (start 118.1755 74.8665) (end 120.015 74.8665) (width 0.25) (layer F.Cu) (net 6))
   (segment (start 120.015 74.909626) (end 122.428 77.322626) (width 0.25) (layer F.Cu) (net 6))
@@
   (segment (start 107.14 73.4895) (end 111.399 73.4895) (width 0.25) (layer F.Cu) (net 32))
   (segment (start 111.399 73.4895) (end 111.633 73.7235) (width 0.25) (layer F.Cu) (net 32))
+  (via (at 138.2395 78.9305) (size 0.8) (drill 0.4) (layers F.Cu B.Cu) (net 34))
   (segment (start 137.958 79.212) (end 138.2395 78.9305) (width 0.25) (layer F.Cu) (net 34))
   (segment (start 137.958 80.529) (end 137.958 79.212) (width 0.25) (layer F.Cu) (net 34))
@@
   (segment (start 164.719 77.6605) (end 164.15852 78.22098) (width 0.25) (layer B.Cu) (net 34))
   (segment (start 168.3385 77.6605) (end 164.719 77.6605) (width 0.25) (layer B.Cu) (net 34))
+  (via (at 140.7795 78.74) (size 0.8) (drill 0.4) (layers F.Cu B.Cu) (net 35))
   (segment (start 140.307388 78.74) (end 140.7795 78.74) (width 0.25) (layer F.Cu) (net 35))
   (segment (start 139.458 79.589388) (end 140.307388 78.74) (width 0.25) (layer F.Cu) (net 35))
@@
   (segment (start 163.70851 77.21049) (end 164.338 76.581) (width 0.25) (layer B.Cu) (net 35))
   (segment (start 164.338 76.581) (end 168.021 76.581) (width 0.25) (layer B.Cu) (net 35))
+  (via (at 167.0685 79.6925) (size 0.8) (drill 0.4) (layers F.Cu B.Cu) (net 36))
+  (via (at 166.3065 75.438) (size 0.8) (drill 0.4) (layers F.Cu B.Cu) (net 36))
+  (via (at 135.763 82.042) (size 0.8) (drill 0.4) (layers F.Cu B.Cu) (net 36))
   (segment (start 136.458 81.347) (end 135.763 82.042) (width 0.25) (layer F.Cu) (net 36))
   (segment (start 136.458 80.529) (end 136.458 81.347) (width 0.25) (layer F.Cu) (net 36))
@@
   (segment (start 163.2585 75.2475) (end 165.227 73.279) (width 0.25) (layer B.Cu) (net 37))
   (segment (start 165.227 73.279) (end 168.402 73.279) (width 0.25) (layer B.Cu) (net 37))
+  (via (at 165.862 79.6925) (size 0.8) (drill 0.4) (layers F.Cu B.Cu) (net 38))
+  (via (at 165.354 71.0565) (size 0.8) (drill 0.4) (layers F.Cu B.Cu) (net 38))
+  (via (at 136.9695 82.169) (size 0.8) (drill 0.4) (layers F.Cu B.Cu) (net 38))
   (segment (start 136.958 82.1575) (end 136.9695 82.169) (width 0.25) (layer F.Cu) (net 38))
   (segment (start 136.958 80.529) (end 136.958 82.1575) (width 0.25) (layer F.Cu) (net 38))
@@
   (segment (start 165.862 78.8035) (end 165.354 78.2955) (width 0.25) (layer F.Cu) (net 38))
   (segment (start 165.354 71.0565) (end 168.3385 71.0565) (width 0.25) (layer B.Cu) (net 38))
+  (via (at 164.719 79.6925) (size 0.8) (drill 0.4) (layers F.Cu B.Cu) (net 39))
+  (via (at 164.1475 70.0405) (size 0.8) (drill 0.4) (layers F.Cu B.Cu) (net 39))
+  (via (at 136.779 78.9305) (size 0.8) (drill 0.4) (layers F.Cu B.Cu) (net 39))
   (segment (start 164.719 79.6925) (end 164.719 72.136) (width 0.25) (layer F.Cu) (net 39))
   (segment (start 164.1475 71.5645) (end 164.1475 70.0405) (width 0.25) (layer F.Cu) (net 39))
