File: eurorack_to_3v3/3v3_to_cv.kicad_sch (KiCad schematic)
At the start: 17 parts, among them U2 TL074CDT, U3 LM324

Commit message: update schematic for eurorack_to_3v, add BH2227 pcb layout
Parts:
- U2, U3: symbol Device:Opamp_Quad_Generic -> Device:Opamp_Quad
Connections:
- net +12V: now also U2.4 (V+), U3.4 (V+)
- net -12V: now also U2.11 (V-), U3.11 (V-)
- net CV_3V3_1: now also U2.3 (+)
- net CV_3V3_2: now also U2.5 (+)
- net CV_3V3_3: now also U2.10 (+)
- net CV_3V3_4: now also U2.12 (+)
- net CV_BIAS: now also U3.1, U3.2 (-)
- net CV_OUT_1: now also U2.1
- net CV_OUT_2: now also U2.7
- net CV_OUT_3: now also U2.8
- net CV_OUT_4: now also U2.14
- net at C1.1, R17.2, R18.1: now also U3.3 (+)
- net at C2.2, R19.2, R21.2: now also U2.2 (-)
- net at C3.2, R20.2, R22.2: now also U2.9 (-)
- net at C4.2, R23.2, R25.2: now also U2.6 (-)
- net at C5.2, R24.2, R26.2: now also U2.13 (-)
Changed lines of the file:
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@@
     (pin "1")
   )
-  (symbol (lib_id "Device:Opamp_Quad_Generic") (at 146.05 86.36 0) (unit 1)
-    (in_bom yes) (on_board yes)
-    (property "Reference" "U2" (id 0) (at 147.32 77.47 0))
-    (property "Value" "TL074CDT" (id 1) (at 147.32 80.01 0))
+  (symbol (lib_id "Device:Opamp_Quad") (at 146.05 86.36 0) (mirror x) (unit 1)
+    (in_bom yes) (on_board yes)
+    (property "Reference" "U2" (id 0) (at 147.32 95.25 0))
+    (property "Value" "TL074CDT" (id 1) (at 147.32 92.71 0))
     (property "Footprint" "Package_SO:SOIC-14_3.9x8.7mm_P1.27mm" (id 2) (at 146.05 86.36 0)
       (effects (font (size 1.27 1.27)) hide)
@@
       (effects (font (size 1.27 1.27)) hide)
     )
+    (pin "1")
+    (pin "2")
+    (pin "3")
   )
   (symbol (lib_id "Device:C") (at 144.78 73.66 270) (unit 1)
@@
     (pin "2")
   )
-  (symbol (lib_id "Device:Opamp_Quad_Generic") (at 63.5 130.81 0) (unit 1)
+  (symbol (lib_id "Device:Opamp_Quad") (at 63.5 130.81 0) (unit 1)
     (in_bom yes) (on_board yes)
     (property "Reference" "U3" (id 0) (at 66.04 125.73 0))
@@
       (effects (font (size 1.27 1.27)) hide)
     )
+    (pin "1")
+    (pin "2")
+    (pin "3")
   )
   (symbol (lib_id "Device:C") (at 144.78 129.54 270) (unit 1)
@@
     (pin "2")
   )
-  (symbol (lib_id "Device:Opamp_Quad_Generic") (at 146.05 142.24 0) (unit 3)
-    (in_bom yes) (on_board yes)
-    (property "Reference" "U2" (id 0) (at 147.32 133.35 0))
-    (property "Value" "TL074CDT" (id 1) (at 147.32 135.89 0))
+  (symbol (lib_id "Device:Opamp_Quad") (at 146.05 142.24 0) (mirror x) (unit 3)
+    (in_bom yes) (on_board yes)
+    (property "Reference" "U2" (id 0) (at 147.32 151.13 0))
+    (property "Value" "TL074CDT" (id 1) (at 147.32 148.59 0))
     (property "Footprint" "Package_SO:SOIC-14_3.9x8.7mm_P1.27mm" (id 2) (at 146.05 142.24 0)
       (effects (font (size 1.27 1.27)) hide)
@@
       (effects (font (size 1.27 1.27)) hide)
     )
+    (pin "10")
+    (pin "8")
+    (pin "9")
   )
   (symbol (lib_id "Device:C") (at 232.41 71.12 270) (unit 1)
@@
     (pin "2")
   )
-  (symbol (lib_id "Device:Opamp_Quad_Generic") (at 233.68 83.82 0) (unit 2)
-    (in_bom yes) (on_board yes)
-    (property "Reference" "U2" (id 0) (at 234.95 74.93 0))
-    (property "Value" "TL074CDT" (id 1) (at 234.95 77.47 0))
+  (symbol (lib_id "Device:Opamp_Quad") (at 233.68 83.82 0) (mirror x) (unit 2)
+    (in_bom yes) (on_board yes)
+    (property "Reference" "U2" (id 0) (at 234.95 92.71 0))
+    (property "Value" "TL074CDT" (id 1) (at 234.95 90.17 0))
     (property "Footprint" "Package_SO:SOIC-14_3.9x8.7mm_P1.27mm" (id 2) (at 233.68 83.82 0)
       (effects (font (size 1.27 1.27)) hide)
@@
       (effects (font (size 1.27 1.27)) hide)
     )
+    (pin "5")
+    (pin "6")
+    (pin "7")
   )
   (symbol (lib_id "Device:C") (at 232.41 127 270) (unit 1)
@@
     (pin "2")
   )
-  (symbol (lib_id "Device:Opamp_Quad_Generic") (at 233.68 139.7 0) (unit 4)
-    (in_bom yes) (on_board yes)
-    (property "Reference" "U2" (id 0) (at 234.95 130.81 0))
-    (property "Value" "TL074CDT" (id 1) (at 234.95 133.35 0))
+  (symbol (lib_id "Device:Opamp_Quad") (at 233.68 139.7 0) (mirror x) (unit 4)
+    (in_bom yes) (on_board yes)
+    (property "Reference" "U2" (id 0) (at 234.95 148.59 0))
+    (property "Value" "TL074CDT" (id 1) (at 234.95 146.05 0))
     (property "Footprint" "Package_SO:SOIC-14_3.9x8.7mm_P1.27mm" (id 2) (at 233.68 139.7 0)
       (effects (font (size 1.27 1.27)) hide)
@@
       (effects (font (size 1.27 1.27)) hide)
     )
-  )
-  (symbol (lib_id "Device:Opamp_Quad_Generic") (at 62.865 167.64 0) (unit 5)
+    (pin "12")
+    (pin "13")
+    (pin "14")
+  )
+  (symbol (lib_id "Device:Opamp_Quad") (at 62.865 167.64 0) (unit 5)
     (in_bom yes) (on_board yes)
     (property "Reference" "U3" (id 0) (at 65.405 162.56 0))
@@
       (effects (font (size 1.27 1.27)) hide)
     )
+    (pin "11")
+    (pin "4")
   )
   (symbol (lib_id "power:+12V") (at 60.325 160.02 0) (unit 1)
@@
     (pin "1")
   )
-  (symbol (lib_id "Device:Opamp_Quad_Generic") (at 187.325 111.125 0) (unit 5)
+  (symbol (lib_id "Device:Opamp_Quad") (at 187.325 111.125 0) (unit 5)
     (in_bom yes) (on_board yes)
     (property "Reference" "U2" (id 0) (at 188.595 109.855 0))
@@
       (effects (font (size 1.27 1.27)) hide)
     )
+    (pin "11")
+    (pin "4")
   )
   (symbol (lib_id "power:-12V") (at 184.785 118.745 180) (unit 1)

Commit message: finished Big One Little One v2
Parts:
- renumbered C1 to C17, C2 to C18, C3 to C19, C4 to C20, C5 to C21, R17 to R55, R18 to R56, R21 to R57, R20 to R58, R19 to R59, R22 to R60, R23 to R61, R24 to R62, R25 to R63, R26 to R64, U2 to U23
Changed lines of the file:
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@@
   (symbol (lib_id "Device:R_US") (at 27.94 121.92 0) (unit 1)
     (in_bom yes) (on_board yes)
-    (property "Reference" "R17" (id 0) (at 29.6672 120.7516 0)
+    (property "Reference" "R55" (id 0) (at 29.6672 120.7516 0)
       (effects (font (size 1.27 1.27)) (justify left))
     )
@@
   (symbol (lib_id "Device:R_US") (at 27.94 135.89 0) (unit 1)
     (in_bom yes) (on_board yes)
-    (property "Reference" "R18" (id 0) (at 29.6672 134.7216 0)
+    (property "Reference" "R56" (id 0) (at 29.6672 134.7216 0)
       (effects (font (size 1.27 1.27)) (justify left))
     )
@@
   (symbol (lib_id "Device:C") (at 41.91 135.89 0) (unit 1)
     (in_bom yes) (on_board yes)
-    (property "Reference" "C1" (id 0) (at 44.831 134.7216 0)
+    (property "Reference" "C17" (id 0) (at 44.831 134.7216 0)
       (effects (font (size 1.27 1.27)) (justify left))
     )
@@
   (symbol (lib_id "power:+12V") (at 27.94 113.03 0) (unit 1)
     (in_bom yes) (on_board yes)
-    (property "Reference" "#PWR08" (id 0) (at 27.94 116.84 0)
+    (property "Reference" "#PWR085" (id 0) (at 27.94 116.84 0)
       (effects (font (size 1.27 1.27)) hide)
     )
@@
   (symbol (lib_id "power:GND") (at 27.94 146.05 0) (unit 1)
     (in_bom yes) (on_board yes)
-    (property "Reference" "#PWR09" (id 0) (at 27.94 152.4 0)
+    (property "Reference" "#PWR086" (id 0) (at 27.94 152.4 0)
       (effects (font (size 1.27 1.27)) hide)
     )
@@
   (symbol (lib_id "power:GND") (at 41.91 146.05 0) (unit 1)
     (in_bom yes) (on_board yes)
-    (property "Reference" "#PWR010" (id 0) (at 41.91 152.4 0)
+    (property "Reference" "#PWR087" (id 0) (at 41.91 152.4 0)
       (effects (font (size 1.27 1.27)) hide)
     )
@@
   (symbol (lib_id "Device:Opamp_Quad") (at 146.05 86.36 0) (mirror x) (unit 1)
     (in_bom yes) (on_board yes)
-    (property "Reference" "U2" (id 0) (at 147.32 95.25 0))
+    (property "Reference" "U23" (id 0) (at 147.32 95.25 0))
     (property "Value" "TL074CDT" (id 1) (at 147.32 92.71 0))
     (property "Footprint" "Package_SO:SOIC-14_3.9x8.7mm_P1.27mm" (id 2) (at 146.05 86.36 0)
@@
   (symbol (lib_id "Device:C") (at 144.78 73.66 270) (unit 1)
     (in_bom yes) (on_board yes)
-    (property "Reference" "C2" (id 0) (at 144.78 67.2592 90))
+    (property "Reference" "C18" (id 0) (at 144.78 67.2592 90))
     (property "Value" "1nF" (id 1) (at 144.78 69.5706 90))
     (property "Footprint" "Capacitor_SMD:C_0402_1005Metric" (id 2) (at 140.97 74.6252 0)
@@
   (symbol (lib_id "Device:R_US") (at 144.78 63.5 270) (unit 1)
     (in_bom yes) (on_board yes)
-    (property "Reference" "R19" (id 0) (at 144.78 58.293 90))
+    (property "Reference" "R59" (id 0) (at 144.78 58.293 90))
     (property "Value" "24K" (id 1) (at 144.78 60.6044 90))
     (property "Footprint" "Resistor_SMD:R_1206_3216Metric" (id 2) (at 144.526 64.516 90)
@@
   (symbol (lib_id "Device:R_US") (at 129.54 83.82 90) (unit 1)
     (in_bom yes) (on_board yes)
-    (property "Reference" "R21" (id 0) (at 129.54 78.613 90))
+    (property "Reference" "R57" (id 0) (at 129.54 78.613 90))
     (property "Value" "11K" (id 1) (at 129.54 80.9244 90))
     (property "Footprint" "Resistor_SMD:R_0402_1005Metric" (id 2) (at 129.794 82.804 90)
@@
   (symbol (lib_id "Device:C") (at 144.78 129.54 270) (unit 1)
     (in_bom yes) (on_board yes)
-    (property "Reference" "C3" (id 0) (at 144.78 123.1392 90))
+    (property "Reference" "C19" (id 0) (at 144.78 123.1392 90))
     (property "Value" "1nF" (id 1) (at 144.78 125.4506 90))
     (property "Footprint" "Capacitor_SMD:C_0402_1005Metric" (id 2) (at 140.97 130.5052 0)
@@
   (symbol (lib_id "Device:R_US") (at 144.78 119.38 270) (unit 1)
     (in_bom yes) (on_board yes)
-    (property "Reference" "R22" (id 0) (at 144.78 114.173 90))
+    (property "Reference" "R60" (id 0) (at 144.78 114.173 90))
     (property "Value" "24K" (id 1) (at 144.78 116.4844 90))
     (property "Footprint" "Resistor_SMD:R_1206_3216Metric" (id 2) (at 144.526 120.396 90)
@@
   (symbol (lib_id "Device:R_US") (at 129.54 139.7 90) (unit 1)
     (in_bom yes) (on_board yes)
-    (property "Reference" "R20" (id 0) (at 129.54 134.493 90))
+    (property "Reference" "R58" (id 0) (at 129.54 134.493 90))
     (property "Value" "11K" (id 1) (at 129.54 136.8044 90))
     (property "Footprint" "Resistor_SMD:R_0402_1005Metric" (id 2) (at 129.794 138.684 90)
@@
   (symbol (lib_id "Device:Opamp_Quad") (at 146.05 142.24 0) (mirror x) (unit 3)
     (in_bom yes) (on_board yes)
-    (property "Reference" "U2" (id 0) (at 147.32 151.13 0))
+    (property "Reference" "U23" (id 0) (at 147.32 151.13 0))
     (property "Value" "TL074CDT" (id 1) (at 147.32 148.59 0))
     (property "Footprint" "Package_SO:SOIC-14_3.9x8.7mm_P1.27mm" (id 2) (at 146.05 142.24 0)
@@
   (symbol (lib_id "Device:C") (at 232.41 71.12 270) (unit 1)
     (in_bom yes) (on_board yes)
-    (property "Reference" "C4" (id 0) (at 232.41 64.7192 90))
+    (property "Reference" "C20" (id 0) (at 232.41 64.7192 90))
     (property "Value" "1nF" (id 1) (at 232.41 67.0306 90))
     (property "Footprint" "Capacitor_SMD:C_0402_1005Metric" (id 2) (at 228.6 72.0852 0)
@@
   (symbol (lib_id "Device:R_US") (at 232.41 60.96 270) (unit 1)
     (in_bom yes) (on_board yes)
-    (property "Reference" "R25" (id 0) (at 232.41 55.753 90))
+    (property "Reference" "R63" (id 0) (at 232.41 55.753 90))
     (property "Value" "24K" (id 1) (at 232.41 58.0644 90))
     (property "Footprint" "Resistor_SMD:R_1206_3216Metric" (id 2) (at 232.156 61.976 90)
@@
   (symbol (lib_id "Device:R_US") (at 217.17 81.28 90) (unit 1)
     (in_bom yes) (on_board yes)
-    (property "Reference" "R23" (id 0) (at 217.17 76.073 90))
+    (property "Reference" "R61" (id 0) (at 217.17 76.073 90))
     (property "Value" "11K" (id 1) (at 217.17 78.3844 90))
     (property "Footprint" "Resistor_SMD:R_0402_1005Metric" (id 2) (at 217.424 80.264 90)
@@
   (symbol (lib_id "Device:Opamp_Quad") (at 233.68 83.82 0) (mirror x) (unit 2)
     (in_bom yes) (on_board yes)
-    (property "Reference" "U2" (id 0) (at 234.95 92.71 0))
+    (property "Reference" "U23" (id 0) (at 234.95 92.71 0))
     (property "Value" "TL074CDT" (id 1) (at 234.95 90.17 0))
     (property "Footprint" "Package_SO:SOIC-14_3.9x8.7mm_P1.27mm" (id 2) (at 233.68 83.82 0)
@@
   (symbol (lib_id "Device:C") (at 232.41 127 270) (unit 1)
     (in_bom yes) (on_board yes)
-    (property "Reference" "C5" (id 0) (at 232.41 120.5992 90))
+    (property "Reference" "C21" (id 0) (at 232.41 120.5992 90))
     (property "Value" "1nF" (id 1) (at 232.41 122.9106 90))
     (property "Footprint" "Capacitor_SMD:C_0402_1005Metric" (id 2) (at 228.6 127.9652 0)
@@
   (symbol (lib_id "Device:R_US") (at 232.41 116.84 270) (unit 1)
     (in_bom yes) (on_board yes)
-    (property "Reference" "R26" (id 0) (at 232.41 111.633 90))
+    (property "Reference" "R64" (id 0) (at 232.41 111.633 90))
     (property "Value" "24K" (id 1) (at 232.41 113.9444 90))
     (property "Footprint" "Resistor_SMD:R_1206_3216Metric" (id 2) (at 232.156 117.856 90)
@@
   (symbol (lib_id "Device:R_US") (at 217.17 137.16 90) (unit 1)
     (in_bom yes) (on_board yes)
-    (property "Reference" "R24" (id 0) (at 217.17 131.953 90))
+    (property "Reference" "R62" (id 0) (at 217.17 131.953 90))
     (property "Value" "11K" (id 1) (at 217.17 134.2644 90))
     (property "Footprint" "Resistor_SMD:R_0402_1005Metric" (id 2) (at 217.424 136.144 90)
@@
   (symbol (lib_id "Device:Opamp_Quad") (at 233.68 139.7 0) (mirror x) (unit 4)
     (in_bom yes) (on_board yes)
-    (property "Reference" "U2" (id 0) (at 234.95 148.59 0))
+    (property "Reference" "U23" (id 0) (at 234.95 148.59 0))
     (property "Value" "TL074CDT" (id 1) (at 234.95 146.05 0))
     (property "Footprint" "Package_SO:SOIC-14_3.9x8.7mm_P1.27mm" (id 2) (at 233.68 139.7 0)
@@
   (symbol (lib_id "power:+12V") (at 60.325 160.02 0) (unit 1)
     (in_bom yes) (on_board yes)
-    (property "Reference" "#PWR040" (id 0) (at 60.325 163.83 0)
+    (property "Reference" "#PWR088" (id 0) (at 60.325 163.83 0)
       (effects (font (size 1.27 1.27)) hide)
     )
@@
   (symbol (lib_id "power:-12V") (at 60.325 175.26 180) (unit 1)
     (in_bom yes) (on_board yes)
-    (property "Reference" "#PWR083" (id 0) (at 60.325 177.8 0)
+    (property "Reference" "#PWR089" (id 0) (at 60.325 177.8 0)
       (effects (font (size 1.27 1.27)) hide)
     )
@@
   (symbol (lib_id "Device:Opamp_Quad") (at 187.325 111.125 0) (unit 5)
     (in_bom yes) (on_board yes)
-    (property "Reference" "U2" (id 0) (at 188.595 109.855 0))
+    (property "Reference" "U23" (id 0) (at 188.595 109.855 0))
     (property "Value" "TL074CDT" (id 1) (at 191.77 112.395 0))
     (property "Footprint" "Package_SO:SOIC-14_3.9x8.7mm_P1.27mm" (id 2) (at 187.325 111.125 0)
@@
   (symbol (lib_id "power:-12V") (at 184.785 118.745 180) (unit 1)
     (in_bom yes) (on_board yes)
-    (property "Reference" "#PWR085" (id 0) (at 184.785 121.285 0)
+    (property "Reference" "#PWR091" (id 0) (at 184.785 121.285 0)
       (effects (font (size 1.27 1.27)) hide)
     )
@@
   (symbol (lib_id "power:+12V") (at 184.785 103.505 0) (unit 1)
     (in_bom yes) (on_board yes)
-    (property "Reference" "#PWR084" (id 0) (at 184.785 107.315 0)
-      (effects (font (size 1.27 1.27)) hide)
-    )
+    (property "Reference" "#PWR090" (id 0) (at 184.785 107.315 0)
+      (effects (font (size 1.27 1.27)) hide)
+    )
