File: eurorack_to_3v3/cv_to_3v3.kicad_sch (KiCad schematic)
At the start: 21 parts, among them U4 MCP6009

Commit message: finished Big One Little One v2
Parts:
- U9: renamed from U4; symbol Device:Opamp_Quad_Generic -> Device:Opamp_Quad
- renumbered C6 to C13, C7 to C14, C8 to C15, C9 to C16, R27 to R19, R28 to R20, R29 to R21, R30 to R22, R31 to R23, R32 to R24, R33 to R25, R34 to R26, R35 to R27, R36 to R28, R37 to R29, R38 to R30
Connections:
- net GND: now also U9.3 (+), U9.3 (+), U9.3 (+), U9.3 (+)
- net cv_3v3_1: now also U9.1
- net cv_3v3_2: now also U9.1
- net cv_3v3_3: now also U9.1
- net cv_3v3_4: now also U9.1
- net at C13.2, R19.1, R20.2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: now also U9.2 (-)
- net at C15.2, R25.1, R26.2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: now also U9.2 (-)
- net at C14.2, R21.1, R22.2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: now also U9.2 (-)
- net at C16.2, R27.1, R28.2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: now also U9.2 (-)
