File: eurorack_to_3v3/eurorack_to_3v3.kicad_pcb (KiCad board)
At the start: 2 copper layers, 47.5 x 96 mm, 154 parts, among them J1 cv_in_2, J2 gate_in_2, J25 Eurorack Power Header, J3 gate_in_1, J30 Brain Bus, J4 cv_in_1, J5 gate_in_3, J6 gate_out, J7 cv_out, U1 LM324, U10 MOSFET_RK7002BM, U11 MOSFET_RK7002BM, U12 MOSFET_RK7002BM, U13 MOSFET_RK7002BM, U14 74HC165, U15 MCP3208, U17 74HC165, U18 74HC137, U19 BH2227FV, U2 TL074CDT, U20 74HC595, U21 MOSFET_RK7002BM, U22 MOSFET_RK7002BM, U23 MOSFET_RK7002BM, U24 MOSFET_RK7002BM, U3 LM324, U4 MCP6009, U5 MOSFET_RK7002BM, U6 MOSFET_RK7002BM, U7 MOSFET_RK7002BM, U8 MOSFET_RK7002BM, U9 MCP6009

Commit message: pcb refactor in progress
Parts:
- removed C15, C16: 22uF, Capacitor_SMD:C_0805_2012Metric
- removed G***: LOGO, ASMR_footprints:SilkScreen_asmrrrrrrrrr
- removed G***: LOGO, ASMR_footprints:Silkscreen_mesh
- removed R39, R40, R45, R46, R63, R64, R69, R70, R77, R78, R83, R84: 100K, Resistor_SMD:R_0805_2012Metric
- removed U14, U17: 74HC165, Package_SO:SOIC-16_3.9x9.9mm_P1.27mm
- U4, U9: value MCP6009 -> 74HC589; footprint Package_SO:SOIC-14_3.9x8.7mm_P1.27mm -> Package_SO:SOIC-16_3.9x9.9mm_P1.27mm
- moved U9 28.2 mm to (153.4, 92.9), turned to 0 degrees
- moved U4 14.6 mm to (145.0, 92.9), turned to 0 degrees
Connections:
- J30 pad 10: Net-(J30-Pad10) -> /LATCH_GATES
- J30 pad 6: /CS[2] -> /DESELECT
- R41 pad 1: Net-(R39-Pad1) -> /gate_to_3v3_A/GATE_IN_1
- R42 pad 1: Net-(R40-Pad1) -> /gate_to_3v3_A/GATE_IN_3
- R47 pad 1: Net-(R45-Pad1) -> /gate_to_3v3_A/GATE_IN_2
- R48 pad 1: Net-(R46-Pad1) -> /gate_to_3v3_A/GATE_IN_4
- R65 pad 1: Net-(R63-Pad1) -> /gate_to_3v3_B/GATE_IN_1
- R66 pad 1: Net-(R64-Pad1) -> /gate_to_3v3_B/GATE_IN_3
- R71 pad 1: Net-(R69-Pad1) -> /gate_to_3v3_B/GATE_IN_2
- R72 pad 1: Net-(R70-Pad1) -> /gate_to_3v3_B/GATE_IN_4
- R79 pad 1: Net-(R77-Pad1) -> /gate_to_3v3_C/GATE_IN_1
- R80 pad 1: Net-(R78-Pad1) -> /gate_to_3v3_C/GATE_IN_3
- R85 pad 1: Net-(R83-Pad1) -> /gate_to_3v3_C/GATE_IN_2
- R86 pad 1: Net-(R84-Pad1) -> /gate_to_3v3_C/GATE_IN_4
- U10 pad 1: Net-(R63-Pad1) -> /gate_to_3v3_B/GATE_IN_1
- U11 pad 1: Net-(R64-Pad1) -> /gate_to_3v3_B/GATE_IN_3
- U12 pad 1: Net-(R69-Pad1) -> /gate_to_3v3_B/GATE_IN_2
- U13 pad 1: Net-(R70-Pad1) -> /gate_to_3v3_B/GATE_IN_4
- U18 pad 10: Net-(U18-Pad10) -> unconnected-(U18-Pad10)
- U18 pad 11: /GATE_OUT_EN -> unconnected-(U18-Pad11)
- U18 pad 12: /GATE_IN_B_EN -> /GATE_OUT_EN
- U18 pad 13: /GATE_IN_A_EN -> /GATE_IN_EN
- U18 pad 3: /CS[2] -> GNDD
- U18 pad 5: GNDD -> /DESELECT
- U18 pad 7: Net-(U18-Pad7) -> unconnected-(U18-Pad7)
- U18 pad 9: Net-(U18-Pad9) -> unconnected-(U18-Pad9)
- U2 pad 10: Net-(C3-Pad2) -> /3v3_to_cv/CV_3V3_3
- U2 pad 12: Net-(C5-Pad2) -> /3v3_to_cv/CV_3V3_4
- U2 pad 13: /3v3_to_cv/CV_3V3_4 -> Net-(C5-Pad2)
- U2 pad 2: /3v3_to_cv/CV_3V3_1 -> Net-(C2-Pad2)
- U2 pad 3: Net-(C2-Pad2) -> /3v3_to_cv/CV_3V3_1
- U2 pad 5: Net-(C4-Pad2) -> /3v3_to_cv/CV_3V3_2
- U2 pad 6: /3v3_to_cv/CV_3V3_2 -> Net-(C4-Pad2)
- U2 pad 9: /3v3_to_cv/CV_3V3_3 -> Net-(C3-Pad2)
- U20 pad 4: Net-(U20-Pad4) -> unconnected-(U20-Pad4)
- U20 pad 5: Net-(U20-Pad5) -> unconnected-(U20-Pad5)
- U20 pad 6: Net-(U20-Pad6) -> unconnected-(U20-Pad6)
- U20 pad 7: Net-(U20-Pad7) -> unconnected-(U20-Pad7)
- U20 pad 9: Net-(U20-Pad9) -> unconnected-(U20-Pad9)
- U21 pad 1: Net-(R77-Pad1) -> /gate_to_3v3_C/GATE_IN_1
- U22 pad 1: Net-(R78-Pad1) -> /gate_to_3v3_C/GATE_IN_3
- U23 pad 1: Net-(R83-Pad1) -> /gate_to_3v3_C/GATE_IN_2
- U24 pad 1: Net-(R84-Pad1) -> /gate_to_3v3_C/GATE_IN_4
- U4 pad 1: /cv_to_3v3_B/cv_3v3_1 -> /gate_to_3v3_A/GATE_3V3_2
- U4 pad 10: GND -> /GATE_IN_EN
- U4 pad 11: GNDD -> /SCK
- U4 pad 12: GND -> /LATCH_GATES
- U4 pad 13: Net-(C9-Pad2) -> /LOAD_GATES
- U4 pad 14: /cv_to_3v3_B/cv_3v3_4 -> GNDD
- U4 pad 2: Net-(C6-Pad2) -> /gate_to_3v3_A/GATE_3V3_3
- U4 pad 3: GND -> /gate_to_3v3_A/GATE_3V3_4
- U4 pad 4: +3V3 -> /gate_to_3v3_B/GATE_3V3_1
- U4 pad 5: GND -> /gate_to_3v3_B/GATE_3V3_2
- U4 pad 6: Net-(C8-Pad2) -> /gate_to_3v3_B/GATE_3V3_3
- U4 pad 7: /cv_to_3v3_B/cv_3v3_2 -> /gate_to_3v3_B/GATE_3V3_4
- U4 pad 8: /cv_to_3v3_B/cv_3v3_3 -> GNDD
- U4 pad 9: Net-(C7-Pad2) -> Net-(U4-Pad9)
- U5 pad 1: Net-(R39-Pad1) -> /gate_to_3v3_A/GATE_IN_1
- U6 pad 1: Net-(R40-Pad1) -> /gate_to_3v3_A/GATE_IN_3
- U7 pad 1: Net-(R45-Pad1) -> /gate_to_3v3_A/GATE_IN_2
- U8 pad 1: Net-(R46-Pad1) -> /gate_to_3v3_A/GATE_IN_4
- U9 pad 1: /cv_to_3v3_A/cv_3v3_1 -> /gate_to_3v3_C/GATE_3V3_2
- U9 pad 10: GND -> /GATE_IN_EN
- U9 pad 11: GNDD -> /SCK
- U9 pad 12: GND -> /LATCH_GATES
- U9 pad 13: Net-(C13-Pad2) -> /LOAD_GATES
- U9 pad 14: /cv_to_3v3_A/cv_3v3_4 -> Net-(U4-Pad9)
- U9 pad 2: Net-(C10-Pad2) -> /gate_to_3v3_C/GATE_3V3_3
- U9 pad 3: GND -> /gate_to_3v3_C/GATE_3V3_4
- U9 pad 4: +3V3 -> unconnected-(U9-Pad4)
- U9 pad 5: GND -> unconnected-(U9-Pad5)
- U9 pad 6: Net-(C12-Pad2) -> unconnected-(U9-Pad6)
- U9 pad 7: /cv_to_3v3_A/cv_3v3_2 -> unconnected-(U9-Pad7)
- U9 pad 8: /cv_to_3v3_A/cv_3v3_3 -> GNDD
- U9 pad 9: Net-(C11-Pad2) -> /POCI
Routing:
- net /LATCH_GATES: track 0.00 -> 61.3 mm
- net /DESELECT: track 0.00 -> 44.9 mm, vias 0 -> 2
- net /CS[2]: track 42.5 -> 0.00 mm, vias 2 -> 0
- net /gate_to_3v3_C/GATE_IN_1: track 4.45 -> 43.9 mm
- net Net-(R77-Pad1): track 37.5 -> 0.00 mm
- net /gate_to_3v3_B/GATE_IN_1: track 3.79 -> 40.1 mm
- net Net-(R63-Pad1): track 34.4 -> 0.00 mm
- net /gate_to_3v3_C/GATE_IN_2: track 3.99 -> 37.3 mm
- net /gate_to_3v3_A/GATE_IN_1: track 3.69 -> 34.0 mm
- net /gate_to_3v3_B/GATE_IN_2: track 4.19 -> 33.1 mm
- net Net-(R83-Pad1): track 28.7 -> 0.00 mm
- net Net-(R39-Pad1): track 28.3 -> 0.00 mm
- net Net-(R69-Pad1): track 27.0 -> 0.00 mm
- net /gate_to_3v3_C/GATE_IN_3: track 3.94 -> 27.1 mm
- net /LOAD_GATES: track 81.7 -> 58.8 mm, vias 4 -> 0
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
Commit message: finished Big One Little One v2
Parts:
- added U8: MCP6009, Package_SO:SOIC-14_3.9x8.7mm_P1.27mm, F.Cu at (134.3, 72.1)
- added U9: MCP6009, Package_SO:SOIC-14_3.9x8.7mm_P1.27mm, F.Cu at (132.3, 85.6)
- renumbered C14 to C1, C11 to C10, C12 to C11, C13 to C12, C6 to C13, C7 to C14, C8 to C15, C9 to C16, C1 to C17, C2 to C18, C3 to C19, C17 to C2, C4 to C20, C5 to C21, C18 to C3, C19 to C4, C20 to C5, C21 to C6, C22 to C7, C23 to C8, C10 to C9, J25 to J5, J30 to J6, J5 to J7, J6 to J8, J7 to J9, R75 to R1, R54 to R10, R55 to R11, R56 to R12, R57 to R13, R58 to R14, R59 to R15, R60 to R16, R61 to R17, R62 to R18, R27 to R19, R76 to R2, R28 to R20, R29 to R21, R30 to R22, R31 to R23, R32 to R24, R33 to R25, R34 to R26, R35 to R27, R36 to R28, R37 to R29, R89 to R3, R38 to R30, R41 to R31, R42 to R32, R43 to R33, R44 to R34, R47 to R35, R48 to R36, R49 to R37, R50 to R38, R65 to R39, R90 to R4, R66 to R40, R67 to R41, R68 to R42, R71 to R43, R72 to R44, R73 to R45, R74 to R46, R79 to R47, R80 to R48, R81 to R49, R91 to R5, R82 to R50, R85 to R51, R86 to R52, R87 to R53, R88 to R54, R17 to R55, R18 to R56, R21 to R57, R20 to R58, R19 to R59, R92 to R6, R22 to R60, R23 to R61, R24 to R62, R25 to R63, R26 to R64, R1 to R65, R2 to R66, R3 to R67, R4 to R68, R5 to R69, R51 to R7, R6 to R70, R7 to R71, R8 to R72, R9 to R73, R10 to R74, R11 to R75, R12 to R76, R13 to R77, R14 to R78, R15 to R79, R52 to R8, R16 to R80, R53 to R9, U15 to U1, U5 to U10, U6 to U11, U7 to U12, U8 to U13, U10 to U14, U11 to U15, U12 to U16, U13 to U17, U21 to U18, U22 to U19, U4 to U2, U23 to U20, U24 to U21, U2 to U23, U1 to U24, U9 to U4, U18 to U5, U19 to U6, U20 to U7
Routing:
- net Net-(U2-Pad9): track 2.18 -> 33.8 mm, vias 0 -> 2
- net /gate_to_3v3_A/GATE_3V3_4: track 65.1 -> 73.7 mm, vias 4 -> 6
- net +3V3: track 273.2 -> 281.2 mm, vias 18 -> 17
- net /gate_to_3v3_C/GATE_3V3_4: track 49.8 -> 55.5 mm
- net /gate_to_3v3_B/GATE_3V3_2: track 47.8 -> 53.4 mm, vias 3 -> 2
- net /gate_to_3v3_B/GATE_3V3_3: track 49.5 -> 54.8 mm
- net /gate_to_3v3_A/GATE_3V3_3: track 57.3 -> 62.6 mm
- net /gate_to_3v3_B/GATE_3V3_1: track 50.9 -> 55.5 mm, vias 3 -> 2
- net /gate_to_3v3_B/GATE_3V3_4: track 57.1 -> 61.6 mm
- net /GATE_IN_EN: track 19.8 -> 15.3 mm
- net GNDD: track 149.0 -> 153.1 mm, vias 24 -> 26
- net /gate_to_3v3_A/GATE_3V3_2: track 51.7 -> 53.6 mm
- net /gate_to_3v3_C/GATE_3V3_3: track 45.0 -> 46.9 mm
- net /gate_to_3v3_C/GATE_3V3_2: track 43.9 -> 45.7 mm, vias 2 -> 4
- net /AREF_-10V: track 121.7 -> 120.9 mm
Other:
- board text added: "v2"
- board text removed: "v1"
