File: eurorack_to_3v3/eurorack_to_3v3.kicad_sch (KiCad schematic)
At the start: 37 parts, among them J1 cv_in_2, J2 gate_in_2, J25 Eurorack Power Header, J3 gate_in_1, J30 Brain Bus, J4 cv_in_1, J5 gate_in_3, J6 gate_out, J7 cv_out, U14 74HC165, U15 MCP3208, U17 74HC165, U18 74HC137, U19 BH2227FV, U20 74HC595, U3 LM324

Commit message: update schematic for eurorack_to_3v, add BH2227 pcb layout
Connections:
- net GNDD: no longer U18.5 (~{E1})
- net DESELECT: now reaches J30.10
- net DESELECT: now also U18.5 (~{E1})
- no-connect marks 17 -> 16
Other:
- moved on the sheet: J30

Commit message: update eurorack_to_3v3 schematic for v2
Parts:
- removed U14, U17: 74HC165, Package_SO:SOIC-16_3.9x9.9mm_P1.27mm, symbol 74xx:74HC165
- added U? (x2): 74HC589, Package_SO:SOIC-16_3.9x9.9mm_P1.27mm, symbol asmr-kicad:74HC589
Connections:
- net GATE_IN_B_EN is gone; now on net GATE_OUT_EN: U18.12 (~{Y3})
- net +3V3: now also U?.16 (Vcc), U?.16 (Vcc)
- net DESELECT: now also J30.6; no longer J30.10
- net GATE_OUT_EN: no longer U18.11 (~{Y4})
- net GNDD: now also U18.3 (A2), U?.14 (SER), U?.8 (GND), U?.8 (GND)
- net LOAD_GATES: now also U?.13 (~{LOAD}), U?.13 (~{LOAD})
- net POCI: now also U?.9 (Qh)
- net SCK: now also U?.11 (SCLK), U?.11 (SCLK)
- net gate_to_3v3_A/GATE_3V3_1: now also U?.15 (D1)
- net gate_to_3v3_A/GATE_3V3_2: now also U?.1 (D2)
- net gate_to_3v3_A/GATE_3V3_3: now also U?.2 (D3)
- net gate_to_3v3_A/GATE_3V3_4: now also U?.3 (D4)
- net gate_to_3v3_B/GATE_3V3_1: now also U?.4 (D5)
- net gate_to_3v3_B/GATE_3V3_2: now also U?.5 (D6)
- net gate_to_3v3_B/GATE_3V3_3: now also U?.6 (D7)
- net gate_to_3v3_B/GATE_3V3_4: now also U?.7 (D8)
- net gate_to_3v3_C/GATE_3V3_1: now also U?.15 (D1)
- net gate_to_3v3_C/GATE_3V3_2: now also U?.1 (D2)
- net gate_to_3v3_C/GATE_3V3_3: now also U?.2 (D3)
- net gate_to_3v3_C/GATE_3V3_4: now also U?.3 (D4)
- removed net CS[2]: J30.6, U18.3 (A2)
- net GATE_IN_A_EN renamed GATE_IN_EN
- net GATE_IN_EN: now also U?.10 (~{OE}), U?.10 (~{OE})
- new net: U?.14 (SER), U?.9 (Qh)
- new net LATCH_GATES: J30.10, U?.12 (LATCH), U?.12 (LATCH)
- no-connect marks 16 -> 13
Other:
- moved on the sheet: C19, J5

Commit message: finished Big One Little One v2
Parts:
- gave numbers to parts that had none: 2
- renumbered C14 to C1, C17 to C2, C18 to C3, C19 to C4, C20 to C5, C21 to C6, C22 to C7, C23 to C8, C16 to C?, C15 to C?, J25 to J5, J30 to J6, J5 to J7, J6 to J8, J7 to J9, R75 to R1, R76 to R2, R89 to R3, R90 to R4, R91 to R5, R92 to R6, U15 to U1, U18 to U5, U19 to U6, U20 to U7
