File: eurorack_to_3v3/gate_to_3v3.kicad_sch (KiCad schematic)
At the start: 16 parts, among them U21 MOSFET_RK7002BM, U22 MOSFET_RK7002BM, U23 MOSFET_RK7002BM, U24 MOSFET_RK7002BM

Commit message: fix gate_to_3v3 schematic
Parts:
- removed R77, R78, R83, R84: 100K, Resistor_SMD:R_0805_2012Metric, symbol Device:R_US
Connections:
- net GATE_IN_1: now also R79.1, U21.1 (Gate)
- net GATE_IN_2: now also R85.1, U23.1 (Gate)
- net GATE_IN_3: now also R80.1, U22.1 (Gate)
- net GATE_IN_4: now also R86.1, U24.1 (Gate)
Other:
- note added: "Gate To 3V3 Each gate input is a high impedance (100K) input driving an N-Channel MOSFET which converts a pulse of arbitrary voltage to a 3.3V pulse. A pull-down resistor keeps the output low when the MOSTFET is in the open state. Simulation: https://tinyurl.com/y5gbk7v4"
- note removed: "Each gate input is a high impedance (100K) input driving an N-Channel MOSFET which converts a pulse of arbitrary voltage to a 3.3V pulse. A pull-down resistor keeps the output low when the MOSTFET is in the open state. Simulation: https://tinyurl.com/yd53ohy7"
Changed lines of the file:
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@@
-    (stroke (width 0) (type default) (color 0 0 0 0))
-  )
-  (wire (pts (xy 174.625 129.54) (xy 177.165 129.54))
     (stroke (width 0) (type default) (color 0 0 0 0))
   )
@@
     (stroke (width 0) (type default) (color 0 0 0 0))
   )
-  (wire (pts (xy 102.235 128.27) (xy 106.045 128.27))
-    (stroke (width 0) (type default) (color 0 0 0 0))
-  )
   (wire (pts (xy 105.41 78.74) (xy 109.22 78.74))
     (stroke (width 0) (type default) (color 0 0 0 0))
@@
     (stroke (width 0) (type default) (color 0 0 0 0))
   )
-  (wire (pts (xy 184.785 129.54) (xy 188.595 129.54))
-    (stroke (width 0) (type default) (color 0 0 0 0))
-  )
-  (wire (pts (xy 184.15 80.01) (xy 187.96 80.01))
+  (wire (pts (xy 181.61 129.54) (xy 188.595 129.54))
+    (stroke (width 0) (type default) (color 0 0 0 0))
+  )
+  (wire (pts (xy 181.61 80.01) (xy 187.96 80.01))
     (stroke (width 0) (type default) (color 0 0 0 0))
   )
@@
     (stroke (width 0) (type default) (color 0 0 0 0))
   )
-  (wire (pts (xy 91.44 78.74) (xy 93.98 78.74))
+  (wire (pts (xy 99.06 78.74) (xy 105.41 78.74))
     (stroke (width 0) (type default) (color 0 0 0 0))
   )
@@
     (stroke (width 0) (type default) (color 0 0 0 0))
   )
+  (wire (pts (xy 99.06 128.27) (xy 106.045 128.27))
+    (stroke (width 0) (type default) (color 0 0 0 0))
+  )
   (wire (pts (xy 105.41 88.9) (xy 105.41 78.74))
     (stroke (width 0) (type default) (color 0 0 0 0))
   )
-  (wire (pts (xy 173.99 80.01) (xy 176.53 80.01))
-    (stroke (width 0) (type default) (color 0 0 0 0))
-  )
-  (wire (pts (xy 92.075 128.27) (xy 94.615 128.27))
-    (stroke (width 0) (type default) (color 0 0 0 0))
-  )
   (wire (pts (xy 200.66 87.63) (xy 210.82 87.63))
     (stroke (width 0) (type default) (color 0 0 0 0))
   )
-  (wire (pts (xy 101.6 78.74) (xy 105.41 78.74))
-    (stroke (width 0) (type default) (color 0 0 0 0))
-  )
   (wire (pts (xy 188.595 139.7) (xy 188.595 129.54))
     (stroke (width 0) (type default) (color 0 0 0 0))
   )
-  (text "Each gate input is a high impedance (100K) input\ndriving an N-Channel MOSFET which converts a\npulse of arbitrary voltage to a 3.3V pulse. A pull-down\nresistor keeps the output low when the MOSTFET is\nin the open state.\n\nSimulation:\nhttps://tinyurl.com/yd53ohy7"
+  (text "Gate To 3V3\n\nEach gate input is a high impedance (100K) input\ndriving an N-Channel MOSFET which converts a\npulse of arbitrary voltage to a 3.3V pulse. A pull-down\nresistor keeps the output low when the MOSTFET is\nin the open state.\n\n\nSimulation:\nhttps://tinyurl.com/y5gbk7v4\n"
     (at 16.51 36.83 0)
     (effects (font (size 1.27 1.27)) (justify left bottom))
   )
-  (hierarchical_label "GATE_IN_3" (shape input) (at 92.075 128.27 180)
+  (hierarchical_label "GATE_IN_3" (shape input) (at 99.06 128.27 180)
     (effects (font (size 1.27 1.27)) (justify right))
   )
@@
     (effects (font (size 1.27 1.27)) (justify left))
   )
-  (hierarchical_label "GATE_IN_2" (shape input) (at 173.99 80.01 180)
+  (hierarchical_label "GATE_IN_2" (shape input) (at 181.61 80.01 180)
     (effects (font (size 1.27 1.27)) (justify right))
   )
-  (hierarchical_label "GATE_IN_1" (shape input) (at 91.44 78.74 180)
+  (hierarchical_label "GATE_IN_1" (shape input) (at 99.06 78.74 180)
     (effects (font (size 1.27 1.27)) (justify right))
   )
@@
     (effects (font (size 1.27 1.27)) (justify left))
   )
-  (hierarchical_label "GATE_IN_4" (shape input) (at 174.625 129.54 180)
+  (hierarchical_label "GATE_IN_4" (shape input) (at 181.61 129.54 180)
     (effects (font (size 1.27 1.27)) (justify right))
-  )
-  (symbol (lib_id "Device:R_US") (at 97.79 78.74 270)
-    (in_bom yes) (on_board yes)
-    (property "Reference" "R77" (id 0) (at 97.79 73.533 90))
-    (property "Value" "100K" (id 1) (at 97.79 75.8444 90))
-    (property "Footprint" "Resistor_SMD:R_0805_2012Metric" (id 2) (at 97.536 79.756 90)
-      (effects (font (size 1.27 1.27)) hide)
-    )
-    (property "Datasheet" "~" (id 3) (at 97.79 78.74 0)
-      (effects (font (size 1.27 1.27)) hide)
-    )
-    (property "mpn" "AC0805FR-13100KL" (id 4) (at 97.79 78.74 0)
-      (effects (font (size 1.27 1.27)) hide)
-    )
-    (pin "1")
-    (pin "2")
   )
   (symbol (lib_id "power:GNDD") (at 118.11 96.52 0)
@@
     (pin "1")
   )
-  (symbol (lib_id "Device:R_US") (at 98.425 128.27 270)
-    (in_bom yes) (on_board yes)
-    (property "Reference" "R78" (id 0) (at 98.425 123.063 90))
-    (property "Value" "100K" (id 1) (at 98.425 125.3744 90))
-    (property "Footprint" "Resistor_SMD:R_0805_2012Metric" (id 2) (at 98.171 129.286 90)
-      (effects (font (size 1.27 1.27)) hide)
-    )
-    (property "Datasheet" "~" (id 3) (at 98.425 128.27 0)
-      (effects (font (size 1.27 1.27)) hide)
-    )
-    (property "mpn" "AC0805FR-13100KL" (id 4) (at 98.425 128.27 0)
-      (effects (font (size 1.27 1.27)) hide)
-    )
-    (pin "1")
-    (pin "2")
-  )
   (symbol (lib_id "asmr-kicad:MOSFET_RK7002BM") (at 118.745 128.27 0)
     (in_bom yes) (on_board yes)
@@
     (pin "1")
   )
-  (symbol (lib_id "Device:R_US") (at 180.34 80.01 270)
-    (in_bom yes) (on_board yes)
-    (property "Reference" "R83" (id 0) (at 180.34 74.803 90))
-    (property "Value" "100K" (id 1) (at 180.34 77.1144 90))
-    (property "Footprint" "Resistor_SMD:R_0805_2012Metric" (id 2) (at 180.086 81.026 90)
-      (effects (font (size 1.27 1.27)) hide)
-    )
-    (property "Datasheet" "~" (id 3) (at 180.34 80.01 0)
-      (effects (font (size 1.27 1.27)) hide)
-    )
-    (property "mpn" "AC0805FR-13100KL" (id 4) (at 180.34 80.01 0)
-      (effects (font (size 1.27 1.27)) hide)
-    )
-    (pin "1")
-    (pin "2")
-  )
   (symbol (lib_id "asmr-kicad:MOSFET_RK7002BM") (at 200.66 80.01 0)
     (in_bom yes) (on_board yes)
@@
     (pin "1")
   )
-  (symbol (lib_id "Device:R_US") (at 180.975 129.54 270)
-    (in_bom yes) (on_board yes)
-    (property "Reference" "R84" (id 0) (at 180.975 124.333 90))
-    (property "Value" "100K" (id 1) (at 180.975 126.6444 90))
-    (property "Footprint" "Resistor_SMD:R_0805_2012Metric" (id 2) (at 180.721 130.556 90)
-      (effects (font (size 1.27 1.27)) hide)
-    )
-    (property "Datasheet" "~" (id 3) (at 180.975 129.54 0)
-      (effects (font (size 1.27 1.27)) hide)
-    )
-    (property "mpn" "AC0805FR-13100KL" (id 4) (at 180.975 129.54 0)
-      (effects (font (size 1.27 1.27)) hide)
-    )
-    (pin "1")
-    (pin "2")
-  )
   (symbol (lib_id "asmr-kicad:MOSFET_RK7002BM") (at 201.295 129.54 0)

Commit message: finished Big One Little One v2
Parts:
- renumbered R79 to R47, R80 to R48, R81 to R49, R82 to R50, R85 to R51, R86 to R52, R87 to R53, R88 to R54, U21 to U18, U22 to U19, U23 to U20, U24 to U21
Changed lines of the file:
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@@
   (symbol (lib_id "power:GNDD") (at 118.11 96.52 0)
     (in_bom yes) (on_board yes)
-    (property "Reference" "#PWR074" (id 0) (at 118.11 102.87 0)
+    (property "Reference" "#PWR076" (id 0) (at 118.11 102.87 0)
       (effects (font (size 1.27 1.27)) hide)
     )
@@
   (symbol (lib_id "power:GNDD") (at 105.41 96.52 0)
     (in_bom yes) (on_board yes)
-    (property "Reference" "#PWR071" (id 0) (at 105.41 102.87 0)
+    (property "Reference" "#PWR073" (id 0) (at 105.41 102.87 0)
       (effects (font (size 1.27 1.27)) hide)
     )
@@
   (symbol (lib_id "power:GNDD") (at 187.96 97.79 0)
     (in_bom yes) (on_board yes)
-    (property "Reference" "#PWR077" (id 0) (at 187.96 104.14 0)
+    (property "Reference" "#PWR079" (id 0) (at 187.96 104.14 0)
       (effects (font (size 1.27 1.27)) hide)
     )
@@
   (symbol (lib_id "power:GNDD") (at 200.66 97.79 0)
     (in_bom yes) (on_board yes)
-    (property "Reference" "#PWR080" (id 0) (at 200.66 104.14 0)
+    (property "Reference" "#PWR082" (id 0) (at 200.66 104.14 0)
       (effects (font (size 1.27 1.27)) hide)
     )
@@
   (symbol (lib_id "power:GNDD") (at 106.045 146.05 0)
     (in_bom yes) (on_board yes)
-    (property "Reference" "#PWR072" (id 0) (at 106.045 152.4 0)
+    (property "Reference" "#PWR074" (id 0) (at 106.045 152.4 0)
       (effects (font (size 1.27 1.27)) hide)
     )
@@
   (symbol (lib_id "power:GNDD") (at 118.745 146.05 0)
     (in_bom yes) (on_board yes)
-    (property "Reference" "#PWR076" (id 0) (at 118.745 152.4 0)
+    (property "Reference" "#PWR078" (id 0) (at 118.745 152.4 0)
       (effects (font (size 1.27 1.27)) hide)
     )
@@
   (symbol (lib_id "power:GNDD") (at 188.595 147.32 0)
     (in_bom yes) (on_board yes)
-    (property "Reference" "#PWR078" (id 0) (at 188.595 153.67 0)
+    (property "Reference" "#PWR080" (id 0) (at 188.595 153.67 0)
       (effects (font (size 1.27 1.27)) hide)
     )
@@
   (symbol (lib_id "power:GNDD") (at 201.295 147.32 0)
     (in_bom yes) (on_board yes)
-    (property "Reference" "#PWR082" (id 0) (at 201.295 153.67 0)
+    (property "Reference" "#PWR084" (id 0) (at 201.295 153.67 0)
       (effects (font (size 1.27 1.27)) hide)
     )
@@
   (symbol (lib_id "asmr-kicad:MOSFET_RK7002BM") (at 118.11 78.74 0)
     (in_bom yes) (on_board yes)
-    (property "Reference" "U21" (id 0) (at 120.3452 77.5716 0)
+    (property "Reference" "U18" (id 0) (at 120.3452 77.5716 0)
       (effects (font (size 1.27 1.27)) (justify left))
     )
@@
   (symbol (lib_id "Device:R_US") (at 105.41 92.71 0)
     (in_bom yes) (on_board yes)
-    (property "Reference" "R79" (id 0) (at 100.203 92.71 90))
+    (property "Reference" "R47" (id 0) (at 100.203 92.71 90))
     (property "Value" "100K" (id 1) (at 102.5144 92.71 90))
     (property "Footprint" "Resistor_SMD:R_0805_2012Metric" (id 2) (at 106.426 92.964 90)
@@
   (symbol (lib_id "Device:R_US") (at 118.11 92.71 0)
     (in_bom yes) (on_board yes)
-    (property "Reference" "R81" (id 0) (at 119.8372 91.5416 0)
+    (property "Reference" "R49" (id 0) (at 119.8372 91.5416 0)
       (effects (font (size 1.27 1.27)) (justify left))
     )
@@
   (symbol (lib_id "power:+3.3V") (at 118.11 67.31 0)
     (in_bom yes) (on_board yes)
-    (property "Reference" "#PWR073" (id 0) (at 118.11 71.12 0)
+    (property "Reference" "#PWR075" (id 0) (at 118.11 71.12 0)
       (effects (font (size 1.27 1.27)) hide)
     )
@@
   (symbol (lib_id "asmr-kicad:MOSFET_RK7002BM") (at 118.745 128.27 0)
     (in_bom yes) (on_board yes)
-    (property "Reference" "U22" (id 0) (at 120.9802 127.1016 0)
+    (property "Reference" "U19" (id 0) (at 120.9802 127.1016 0)
       (effects (font (size 1.27 1.27)) (justify left))
     )
@@
   (symbol (lib_id "Device:R_US") (at 106.045 142.24 0)
     (in_bom yes) (on_board yes)
-    (property "Reference" "R80" (id 0) (at 100.838 142.24 90))
+    (property "Reference" "R48" (id 0) (at 100.838 142.24 90))
     (property "Value" "100K" (id 1) (at 103.1494 142.24 90))
     (property "Footprint" "Resistor_SMD:R_0805_2012Metric" (id 2) (at 107.061 142.494 90)
@@
   (symbol (lib_id "Device:R_US") (at 118.745 142.24 0)
     (in_bom yes) (on_board yes)
-    (property "Reference" "R82" (id 0) (at 120.4722 141.0716 0)
+    (property "Reference" "R50" (id 0) (at 120.4722 141.0716 0)
       (effects (font (size 1.27 1.27)) (justify left))
     )
@@
   (symbol (lib_id "power:+3.3V") (at 118.745 116.84 0)
     (in_bom yes) (on_board yes)
-    (property "Reference" "#PWR075" (id 0) (at 118.745 120.65 0)
+    (property "Reference" "#PWR077" (id 0) (at 118.745 120.65 0)
       (effects (font (size 1.27 1.27)) hide)
     )
@@
   (symbol (lib_id "asmr-kicad:MOSFET_RK7002BM") (at 200.66 80.01 0)
     (in_bom yes) (on_board yes)
-    (property "Reference" "U23" (id 0) (at 202.8952 78.8416 0)
+    (property "Reference" "U20" (id 0) (at 202.8952 78.8416 0)
       (effects (font (size 1.27 1.27)) (justify left))
     )
@@
   (symbol (lib_id "Device:R_US") (at 187.96 93.98 0)
     (in_bom yes) (on_board yes)
-    (property "Reference" "R85" (id 0) (at 182.753 93.98 90))
+    (property "Reference" "R51" (id 0) (at 182.753 93.98 90))
     (property "Value" "100K" (id 1) (at 185.0644 93.98 90))
     (property "Footprint" "Resistor_SMD:R_0805_2012Metric" (id 2) (at 188.976 94.234 90)
@@
   (symbol (lib_id "Device:R_US") (at 200.66 93.98 0)
     (in_bom yes) (on_board yes)
-    (property "Reference" "R87" (id 0) (at 202.3872 92.8116 0)
+    (property "Reference" "R53" (id 0) (at 202.3872 92.8116 0)
       (effects (font (size 1.27 1.27)) (justify left))
     )
@@
   (symbol (lib_id "power:+3.3V") (at 200.66 68.58 0)
     (in_bom yes) (on_board yes)
-    (property "Reference" "#PWR079" (id 0) (at 200.66 72.39 0)
+    (property "Reference" "#PWR081" (id 0) (at 200.66 72.39 0)
       (effects (font (size 1.27 1.27)) hide)
     )
@@
   (symbol (lib_id "asmr-kicad:MOSFET_RK7002BM") (at 201.295 129.54 0)
     (in_bom yes) (on_board yes)
-    (property "Reference" "U24" (id 0) (at 203.5302 128.3716 0)
+    (property "Reference" "U21" (id 0) (at 203.5302 128.3716 0)
       (effects (font (size 1.27 1.27)) (justify left))
     )
@@
   (symbol (lib_id "Device:R_US") (at 188.595 143.51 0)
     (in_bom yes) (on_board yes)
-    (property "Reference" "R86" (id 0) (at 183.388 143.51 90))
+    (property "Reference" "R52" (id 0) (at 183.388 143.51 90))
     (property "Value" "100K" (id 1) (at 185.6994 143.51 90))
     (property "Footprint" "Resistor_SMD:R_0805_2012Metric" (id 2) (at 189.611 143.764 90)
@@
   (symbol (lib_id "Device:R_US") (at 201.295 143.51 0)
     (in_bom yes) (on_board yes)
-    (property "Reference" "R88" (id 0) (at 203.0222 142.3416 0)
+    (property "Reference" "R54" (id 0) (at 203.0222 142.3416 0)
       (effects (font (size 1.27 1.27)) (justify left))
     )
@@
   (symbol (lib_id "power:+3.3V") (at 201.295 118.11 0)
     (in_bom yes) (on_board yes)
-    (property "Reference" "#PWR081" (id 0) (at 201.295 121.92 0)
-      (effects (font (size 1.27 1.27)) hide)
-    )
+    (property "Reference" "#PWR083" (id 0) (at 201.295 121.92 0)
+      (effects (font (size 1.27 1.27)) hide)
+    )
