File: at42qt148_captouch/at42qt148_captouch.kicad_pcb (KiCad board)
At the start: 2 copper layers, 74.8 x 26.6 mm, 43 parts, among them IC1 TCR2EF50,LM_CT, IC2 AT42QT1481-ANR, J1 Conn_01x04, J2 Conn_01x04, J3 Conn_01x08, J4 Conn_01x06, Y1 WE_XTAL_830011263_16MHZ

Commit message: finish designing touch sensor dev board
Routing:
- net +5VD: track 10.2 -> 56.5 mm, vias 0 -> 2
- net /Y3A: track 2.40 -> 47.5 mm, vias 0 -> 2
- net /Y2A: track 2.40 -> 46.5 mm, vias 0 -> 2
- net /Y1A: track 2.33 -> 46.1 mm, vias 0 -> 2
- net /Y0A: track 2.38 -> 44.1 mm, vias 0 -> 2
- net +5V: track 43.8 -> 78.2 mm, vias 0 -> 4
- net /Y5A: track 2.45 -> 36.4 mm, vias 0 -> 4
- net /SCOPE_SYNC: track 0.00 -> 33.2 mm, vias 0 -> 2
- net /Y5B: track 4.65 -> 34.9 mm, vias 0 -> 4
- net /Y4A: track 2.45 -> 32.6 mm, vias 0 -> 2
- net /~{DRDY}: track 0.00 -> 29.9 mm, vias 0 -> 2
- net /Y4B: track 4.65 -> 30.2 mm, vias 0 -> 4
- net /SMP: track 26.1 -> 50.0 mm, vias 7 -> 10
- net /Y3B: track 4.57 -> 21.4 mm, vias 0 -> 2
- net /Y2B: track 4.57 -> 21.3 mm, vias 0 -> 2
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Other:
- board text added: "AT42QT Dev Board v1"
