File: high_speed_opamp_sot-23-5_breakout/high_speed_opamp_sot-23-5_breakout.kicad_pcb (KiCad board)
At the start: 2 copper layers, 14.2 x 9.4 mm, 3 parts, among them J1 Conn_01x02_Male, J2 Conn_01x03_Male, U1 LMH6609MF

Commit message: added copper fill to pcb
Routing:
- added copper zone on F.Cu, net (none)
Changed lines of the file:
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@@
     (pad_to_mask_clearance 0)
     (pcbplotparams
-      (layerselection 0x0001000_7fffffff)
+      (layerselection 0x0000000_7fffffff)
       (disableapertmacros false)
       (usegerberextensions false)
@@
   (segment (start 140.618248 92.39) (end 138.2975 92.39) (width 0.25) (layer "F.Cu") (net 5))
   (arc (start 141.765 91.915) (mid 141.238865 92.266551) (end 140.618248 92.39) (width 0.25) (layer "F.Cu") (net 5))
+  (zone (net 0) (net_name "") (layer "F.Cu") (hatch edge 0.508)
+    (connect_pads (clearance 0.508))
+    (min_thickness 0.254) (filled_areas_thickness no)
+    (fill yes (thermal_gap 0.508) (thermal_bridge_width 0.508))
+    (polygon
+      (pts
+        (xy 144.272 96.012)
+        (xy 130.048 96.012)
+        (xy 130.048 86.614)
+        (xy 144.272 86.614)
+      )
+    )
+  )
 )
