File: IQS550_captouch_breakout/IQS550_captouch_breakout.kicad_sch (KiCad schematic)
At the start: 12 parts

Commit message: finished IQS550 pcb
Parts:
- C1, C2, C3, C4, C5, C6: renamed from C?; footprint (none) -> Capacitor_SMD:C_0805_2012Metric
- J2: renamed from J?; footprint (none) -> Connector_PinHeader_2.54mm:PinHeader_1x05_P2.54mm_Vertical
- R1, R2: renamed from R?; footprint (none) -> Resistor_SMD:R_0805_2012Metric
- gave numbers to parts that had none: 3
Connections:
- net +3V3: now also C1.1, C3.1, C5.1, IC1.38 (VDDIO), IC1.7 (VDDHI)
- net GND: now also J3.17, J3.19, J3.21, J3.23, J3.25, J3.27, J3.29, J3.31
- net NRST: now reaches C6.1, IC1.10 (NRST)
- no-connect marks 22 -> 25
Other:
- note added: "PGM and NRST are not needed. "A bootloader is included to allow easy application firmware upgrading via the I2C bus, without the need to access the PGM and NRST pins for reprogramming.""
- note removed: "Question: Where do PGM and SW_IN go?"
