File: captouch_experiments/08_padded_interleaved_loose/08_padded_interleaved_loose.kicad_sch (KiCad schematic)
At the start: 3 parts, among them J1 Conn_01x08_Male, J2 Conn_01x32_Male, U1 captouch_8x32_grid

Commit message: added cap touch padded interleaved sensor boards
Parts:
- U1: footprint ASMR_footprints:captouch_8x32_padded_interleaved -> ASMR_footprints:captouch_8x32_padded_interleaved_loose
Changed lines of the file:
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@@
     (property "Reference" "U1" (id 0) (at 146.05 53.501 0))
     (property "Value" "captouch_8x32_grid" (id 1) (at 146.05 56.0379 0))
-    (property "Footprint" "ASMR_footprints:captouch_8x32_padded_interleaved" (id 2) (at 140.335 57.15 0)
+    (property "Footprint" "ASMR_footprints:captouch_8x32_padded_interleaved_loose" (id 2) (at 140.335 57.15 0)
       (effects (font (size 1.27 1.27)) hide)
     )
@@
     )
     (path "/b6156c27-f6bf-48ba-a852-1e97e3507fa3"
-      (reference "U1") (unit 1) (value "captouch_8x32_grid") (footprint "ASMR_footprints:captouch_8x32_padded_interleaved")
+      (reference "U1") (unit 1) (value "captouch_8x32_grid") (footprint "ASMR_footprints:captouch_8x32_padded_interleaved_loose")
     )
   )
