File: captouch_experiments/14_8x32_self_capacitance/14_8x32_self_capacitance.kicad_pcb (KiCad board)
At the start: 2 copper layers, 218.9 x 80.8 mm, 20 parts, among them J2 Conn_01x16, U1 CD74HC4067M, U10 CD74HC4067M, U11 74HC4051, U12 CD74HC4067M, U13 CD74HC4067M, U14 CD74HC4067M, U15 CD74HC4067M, U16 CD74HC4067M, U17 CD74HC4067M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

Commit message: print 256 self cap touch board and fpc breakout
Other:
- board text added: "8x32 Capacitive Sensor self-mode v2"
- board text removed: "4x16 Capacitive Sensor self-mode v1"
Changed lines of the file:
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@@
   )
   (gr_rect (start 46.3 38.8) (end 265.2 119.6) (layer "Edge.Cuts") (width 0.1) (fill none))
-  (gr_text "4x16 Capacitive Sensor\nself-mode v1" (at 61.775 109.575) (layer "F.SilkS")
+  (gr_text "8x32 Capacitive Sensor\nself-mode v2" (at 61.775 109.575) (layer "F.SilkS")
     (effects (font (size 1 1) (thickness 0.15)) (justify left))
   )
